File: brd/power-supply.sch (KiCad schematic (older format))
At the start: 11 parts, among them J8 POWER, Q1 DMP2040, U4 MC78M05, U5 REF3020

Commit message: corregido problema con referencia analogica
Parts:
- added R27: 220R, Resistors_SMD:R_0805_HandSoldering, symbol R
Connections:
- net VDDA: now also R27.1; no longer U5.2 (OUT)
- new net: R27.2, U5.2 (OUT)
Other:
- moved on the sheet: C14
Changed lines of the file:
@@
 $EndComp
 $Comp
-L GND #PWR030
+L GND #PWR30
 U 1 1 5DA467DA
 P 4050 3600
-F 0 "#PWR030" H 4050 3350 50  0001 C CNN
+F 0 "#PWR30" H 4050 3350 50  0001 C CNN
 F 1 "GND" H 4050 3450 50  0000 C CNN
 F 2 "" H 4050 3600 50  0001 C CNN
@@
 $EndComp
 $Comp
-L +12V #PWR031
+L +12V #PWR31
 U 1 1 5DA467F0
 P 5150 3200
-F 0 "#PWR031" H 5150 3050 50  0001 C CNN
+F 0 "#PWR31" H 5150 3050 50  0001 C CNN
 F 1 "+12V" H 5150 3340 50  0000 C CNN
 F 2 "" H 5150 3200 50  0001 C CNN
@@
 L C C14
 U 1 1 5DA46918
-P 8150 4100
-F 0 "C14" H 8175 4200 50  0000 L CNN
-F 1 "100nF" H 8175 4000 50  0000 L CNN
-F 2 "Capacitors_SMD:C_0805" H 8188 3950 50  0001 C CNN
-F 3 "" H 8150 4100 50  0001 C CNN
-F 4 "Kemet" H 8150 4100 60  0001 C CNN "Manufacturer"
-F 5 "C0805C104J5RACTU" H 8150 4100 60  0001 C CNN "Manufacturer Part Number"
-	1    8150 4100
+P 8525 4100
+F 0 "C14" H 8550 4200 50  0000 L CNN
+F 1 "100nF" H 8550 4000 50  0000 L CNN
+F 2 "Capacitors_SMD:C_0805" H 8563 3950 50  0001 C CNN
+F 3 "" H 8525 4100 50  0001 C CNN
+F 4 "Kemet" H 8525 4100 60  0001 C CNN "Manufacturer"
+F 5 "C0805C104J5RACTU" H 8525 4100 60  0001 C CNN "Manufacturer Part Number"
+	1    8525 4100
 	1    0    0    -1
 $EndComp
@@
 $EndComp
 $Comp
-L +5V #PWR032
+L +5V #PWR36
 U 1 1 5DA46A3A
 P 6600 3200
-F 0 "#PWR032" H 6600 3050 50  0001 C CNN
+F 0 "#PWR36" H 6600 3050 50  0001 C CNN
 F 1 "+5V" H 6600 3340 50  0000 C CNN
 F 2 "" H 6600 3200 50  0001 C CNN
@@
 $EndComp
 $Comp
-L VDDA #PWR033
+L VDDA #PWR41
 U 1 1 5DA46A5C
-P 8150 3650
-F 0 "#PWR033" H 8150 3500 50  0001 C CNN
-F 1 "VDDA" H 8150 3800 50  0000 C CNN
-F 2 "" H 8150 3650 50  0001 C CNN
-F 3 "" H 8150 3650 50  0001 C CNN
-	1    8150 3650
+P 8525 3650
+F 0 "#PWR41" H 8525 3500 50  0001 C CNN
+F 1 "VDDA" H 8525 3800 50  0000 C CNN
+F 2 "" H 8525 3650 50  0001 C CNN
+F 3 "" H 8525 3650 50  0001 C CNN
+	1    8525 3650
 	1    0    0    -1
 $EndComp
@@
 	4050 3450 4050 3600
 $Comp
-L GND #PWR034
+L GND #PWR34
 U 1 1 5DA46D6E
 P 5700 3950
-F 0 "#PWR034" H 5700 3700 50  0001 C CNN
+F 0 "#PWR34" H 5700 3700 50  0001 C CNN
 F 1 "GND" H 5700 3800 50  0000 C CNN
 F 2 "" H 5700 3950 50  0001 C CNN
@@
 	6600 3200 6600 3500
 $Comp
-L GND #PWR035
+L GND #PWR37
 U 1 1 5DA46EC3
 P 6600 3950
-F 0 "#PWR035" H 6600 3700 50  0001 C CNN
+F 0 "#PWR37" H 6600 3700 50  0001 C CNN
 F 1 "GND" H 6600 3800 50  0000 C CNN
 F 2 "" H 6600 3950 50  0001 C CNN
@@
 Connection ~ 6600 3350
 $Comp
-L GND #PWR036
+L GND #PWR35
 U 1 1 5DA46F20
 P 6150 3950
-F 0 "#PWR036" H 6150 3700 50  0001 C CNN
+F 0 "#PWR35" H 6150 3700 50  0001 C CNN
 F 1 "GND" H 6150 3800 50  0000 C CNN
 F 2 "" H 6150 3950 50  0001 C CNN
@@
 	6150 3650 6150 3950
 Wire Wire Line
-	8000 3800 8150 3800
-Wire Wire Line
-	8150 3650 8150 3950
-Connection ~ 8150 3800
+	8375 3800 8525 3800
+Wire Wire Line
+	8525 3650 8525 3950
+Connection ~ 8525 3800
 Wire Wire Line
 	7600 3350 7600 3500
@@
 Connection ~ 6900 3350
 $Comp
-L GND #PWR037
+L GND #PWR42
 U 1 1 5DA47167
-P 8150 4400
-F 0 "#PWR037" H 8150 4150 50  0001 C CNN
-F 1 "GND" H 8150 4250 50  0000 C CNN
-F 2 "" H 8150 4400 50  0001 C CNN
-F 3 "" H 8150 4400 50  0001 C CNN
-	1    8150 4400
-	1    0    0    -1
-$EndComp
-$Comp
-L GND #PWR038
+P 8525 4400
+F 0 "#PWR42" H 8525 4150 50  0001 C CNN
+F 1 "GND" H 8525 4250 50  0000 C CNN
+F 2 "" H 8525 4400 50  0001 C CNN
+F 3 "" H 8525 4400 50  0001 C CNN
+	1    8525 4400
+	1    0    0    -1
+$EndComp
+$Comp
+L GND #PWR40
 U 1 1 5DA47187
 P 7600 4400
-F 0 "#PWR038" H 7600 4150 50  0001 C CNN
+F 0 "#PWR40" H 7600 4150 50  0001 C CNN
 F 1 "GND" H 7600 4250 50  0000 C CNN
 F 2 "" H 7600 4400 50  0001 C CNN
@@
 $EndComp
 Wire Wire Line
-	8150 4400 8150 4250
+	8525 4400 8525 4250
 Wire Wire Line
 	7600 4400 7600 4100
 $Comp
-L GND #PWR039
+L GND #PWR38
 U 1 1 5DA47203
 P 6900 3950
-F 0 "#PWR039" H 6900 3700 50  0001 C CNN
+F 0 "#PWR38" H 6900 3700 50  0001 C CNN
 F 1 "GND" H 6900 3800 50  0000 C CNN
 F 2 "" H 6900 3950 50  0001 C CNN
@@
 $EndComp
 $Comp
-L GND #PWR040
+L GND #PWR33
 U 1 1 5DA475DC
 P 5400 3950
-F 0 "#PWR040" H 5400 3700 50  0001 C CNN
+F 0 "#PWR33" H 5400 3700 50  0001 C CNN
 F 1 "GND" H 5400 3800 50  0000 C CNN
 F 2 "" H 5400 3950 50  0001 C CNN
@@
 $EndComp
 $Comp
-L GND #PWR041
+L GND #PWR32
 U 1 1 5DA47602
 P 5150 3950
-F 0 "#PWR041" H 5150 3700 50  0001 C CNN
+F 0 "#PWR32" H 5150 3700 50  0001 C CNN
 F 1 "GND" H 5150 3800 50  0000 C CNN
 F 2 "" H 5150 3950 50  0001 C CNN
@@
 $EndComp
 $Comp
-L GND #PWR042
+L GND #PWR39
 U 1 1 5DA47D0C
 P 7250 4400
-F 0 "#PWR042" H 7250 4150 50  0001 C CNN
+F 0 "#PWR39" H 7250 4150 50  0001 C CNN
 F 1 "GND" H 7250 4250 50  0000 C CNN
 F 2 "" H 7250 4400 50  0001 C CNN
@@
 	4400 3450 4250 3450
 Connection ~ 4250 3450
+$Comp
+L R R27
+U 1 1 5F2072B2
+P 8225 3800
+F 0 "R27" V 8125 3750 50  0000 C CNN
+F 1 "220R" V 8225 3800 50  0000 C CNN
+F 2 "Resistors_SMD:R_0805_HandSoldering" V 8155 3800 50  0001 C CNN
+F 3 "" H 8225 3800 50  0001 C CNN
+F 4 "Bourns" H 8225 3800 60  0001 C CNN "Manufacturer"
+F 5 "CR0805-JW-221ELF" H 8225 3800 60  0001 C CNN "Manufacturer Part Number"
+	1    8225 3800
+	0    1    1    0
+$EndComp
+Wire Wire Line
+	8000 3800 8075 3800
 $EndSCHEMATC
