File: brd/silent-audio-motion.sch (KiCad schematic (older format))
At the start: 25 parts, among them J1 AUDIO_IN, J2 ISP, J3 UART, J4 OUT_L, J5 OUT_R, U1 MCP6004, U2 ATMEGA328P-AU, U3 TB6612FNG, Y1 16MHz

Commit message: añadido pin DTR para reset en cabecera UART
Parts:
- removed J3: UART, Pin_Headers:Pin_Header_Straight_1x03_Pitch2.54mm, symbol Conn_01x03
- added C17: 100nF, Capacitors_SMD:C_0805, symbol C
- added J3: UART, Pin_Headers:Pin_Header_Straight_1x04_Pitch2.54mm, symbol Conn_01x04
Connections:
- net GND: now also J3.3 (Pin_3)
- net ~RST: now reaches J2.5 (Pin_5), R3.2, U2.29 ((PCINT14/~RESET~)PC6)
- net ~RST: now also C17.2
- net at U2.30 ((PCINT16/RXD)PD0): now also J3.2 (Pin_2)
- net at U2.31 ((PCINT17/TXD)PD1): now also J3.1 (Pin_1)
- new net: C17.1, J3.4 (Pin_4)
Changed lines of the file:
@@
 BPWM
 $Comp
-L GND #PWR14
+L GND #PWR01
 U 1 1 5DA5B0FC
 P 4600 5050
-F 0 "#PWR14" H 4600 4800 50  0001 C CNN
+F 0 "#PWR01" H 4600 4800 50  0001 C CNN
 F 1 "GND" H 4600 4900 50  0000 C CNN
 F 2 "" H 4600 5050 50  0001 C CNN
@@
 $EndComp
 $Comp
-L +5V #PWR11
+L +5V #PWR02
 U 1 1 5DA5B150
 P 4600 2350
-F 0 "#PWR11" H 4600 2200 50  0001 C CNN
+F 0 "#PWR02" H 4600 2200 50  0001 C CNN
 F 1 "+5V" H 4600 2490 50  0000 C CNN
 F 2 "" H 4600 2350 50  0001 C CNN
@@
 $EndComp
 $Comp
-L VDDA #PWR12
+L VDDA #PWR03
 U 1 1 5DA5B1C4
 P 4600 3100
-F 0 "#PWR12" H 4600 2950 50  0001 C CNN
+F 0 "#PWR03" H 4600 2950 50  0001 C CNN
 F 1 "VDDA" H 4600 3250 50  0000 C CNN
 F 2 "" H 4600 3100 50  0001 C CNN
@@
 Connection ~ 4300 2900
 $Comp
-L GND #PWR13
+L GND #PWR04
 U 1 1 5DA5BACE
 P 4600 3700
-F 0 "#PWR13" H 4600 3450 50  0001 C CNN
+F 0 "#PWR04" H 4600 3450 50  0001 C CNN
 F 1 "GND" H 4600 3550 50  0000 C CNN
 F 2 "" H 4600 3700 50  0001 C CNN
@@
 $EndComp
 $Comp
-L GND #PWR10
+L GND #PWR05
 U 1 1 5DA5BB27
 P 4300 3700
-F 0 "#PWR10" H 4300 3450 50  0001 C CNN
+F 0 "#PWR05" H 4300 3450 50  0001 C CNN
 F 1 "GND" H 4300 3550 50  0000 C CNN
 F 2 "" H 4300 3700 50  0001 C CNN
@@
 	4300 3700 4300 3600
 $Comp
-L GND #PWR16
+L GND #PWR06
 U 1 1 5DA5BCF3
 P 5700 2200
-F 0 "#PWR16" H 5700 1950 50  0001 C CNN
+F 0 "#PWR06" H 5700 1950 50  0001 C CNN
 F 1 "GND" H 5700 2050 50  0000 C CNN
 F 2 "" H 5700 2200 50  0001 C CNN
@@
 $EndComp
 $Comp
-L +5V #PWR15
+L +5V #PWR07
 U 1 1 5DA5BD4C
 P 5700 1600
-F 0 "#PWR15" H 5700 1450 50  0001 C CNN
+F 0 "#PWR07" H 5700 1450 50  0001 C CNN
 F 1 "+5V" H 5700 1740 50  0000 C CNN
 F 2 "" H 5700 1600 50  0001 C CNN
@@
 	5700 2050 5700 2200
 $Comp
-L GND #PWR18
+L GND #PWR08
 U 1 1 5DA5C11E
 P 6200 2200
-F 0 "#PWR18" H 6200 1950 50  0001 C CNN
+F 0 "#PWR08" H 6200 1950 50  0001 C CNN
 F 1 "GND" H 6200 2050 50  0000 C CNN
 F 2 "" H 6200 2200 50  0001 C CNN
@@
 $EndComp
 $Comp
-L +5V #PWR17
+L +5V #PWR09
 U 1 1 5DA5C177
 P 6200 1700
-F 0 "#PWR17" H 6200 1550 50  0001 C CNN
+F 0 "#PWR09" H 6200 1550 50  0001 C CNN
 F 1 "+5V" H 6200 1840 50  0000 C CNN
 F 2 "" H 6200 1700 50  0001 C CNN
@@
 $EndComp
 $Comp
-L GND #PWR20
+L GND #PWR010
 U 1 1 5DA5C860
 P 7400 3950
-F 0 "#PWR20" H 7400 3700 50  0001 C CNN
+F 0 "#PWR010" H 7400 3700 50  0001 C CNN
 F 1 "GND" H 7400 3800 50  0000 C CNN
 F 2 "" H 7400 3950 50  0001 C CNN
@@
 $EndComp
 $Comp
-L GND #PWR21
+L GND #PWR011
 U 1 1 5DA5C8B9
 P 7700 3950
-F 0 "#PWR21" H 7700 3700 50  0001 C CNN
+F 0 "#PWR011" H 7700 3700 50  0001 C CNN
 F 1 "GND" H 7700 3800 50  0000 C CNN
 F 2 "" H 7700 3950 50  0001 C CNN
@@
 $EndComp
 $Comp
-L +5V #PWR19
+L +5V #PWR012
 U 1 1 5DA5DC78
 P 7150 1250
-F 0 "#PWR19" H 7150 1100 50  0001 C CNN
+F 0 "#PWR012" H 7150 1100 50  0001 C CNN
 F 1 "+5V" H 7150 1390 50  0000 C CNN
 F 2 "" H 7150 1250 50  0001 C CNN
@@
 	8200 4300 8200 4050
 $Comp
-L GND #PWR22
+L GND #PWR013
 U 1 1 5DA5FD1C
 P 8400 4550
-F 0 "#PWR22" H 8400 4300 50  0001 C CNN
+F 0 "#PWR013" H 8400 4300 50  0001 C CNN
 F 1 "GND" H 8400 4400 50  0000 C CNN
 F 2 "" H 8400 4550 50  0001 C CNN
@@
 Connection ~ 10500 3700
 $Comp
-L GND #PWR24
+L GND #PWR014
 U 1 1 5DA61318
 P 9700 4750
-F 0 "#PWR24" H 9700 4500 50  0001 C CNN
+F 0 "#PWR014" H 9700 4500 50  0001 C CNN
 F 1 "GND" H 9700 4600 50  0000 C CNN
 F 2 "" H 9700 4750 50  0001 C CNN
@@
 Connection ~ 9700 4600
 $Comp
-L +12V #PWR25
+L +12V #PWR015
 U 1 1 5DA61805
 P 9900 2250
-F 0 "#PWR25" H 9900 2100 50  0001 C CNN
+F 0 "#PWR015" H 9900 2100 50  0001 C CNN
 F 1 "+12V" H 9900 2390 50  0000 C CNN
 F 2 "" H 9900 2250 50  0001 C CNN
@@
 $EndComp
 $Comp
-L +5V #PWR23
+L +5V #PWR016
 U 1 1 5DA61935
 P 9500 2250
-F 0 "#PWR23" H 9500 2100 50  0001 C CNN
+F 0 "#PWR016" H 9500 2100 50  0001 C CNN
 F 1 "+5V" H 9500 2390 50  0000 C CNN
 F 2 "" H 9500 2250 50  0001 C CNN
@@
 $EndComp
 $Comp
-L +12V #PWR28
+L +12V #PWR017
 U 1 1 5DA63ADE
 P 10600 1850
-F 0 "#PWR28" H 10600 1700 50  0001 C CNN
+F 0 "#PWR017" H 10600 1700 50  0001 C CNN
 F 1 "+12V" H 10600 1990 50  0000 C CNN
 F 2 "" H 10600 1850 50  0001 C CNN
@@
 $EndComp
 $Comp
-L +5V #PWR26
+L +5V #PWR018
 U 1 1 5DA63B52
 P 10150 1950
-F 0 "#PWR26" H 10150 1800 50  0001 C CNN
+F 0 "#PWR018" H 10150 1800 50  0001 C CNN
 F 1 "+5V" H 10150 2090 50  0000 C CNN
 F 2 "" H 10150 1950 50  0001 C CNN
@@
 $EndComp
 $Comp
-L GND #PWR27
+L GND #PWR019
 U 1 1 5DA63C18
 P 10150 2500
-F 0 "#PWR27" H 10150 2250 50  0001 C CNN
+F 0 "#PWR019" H 10150 2250 50  0001 C CNN
 F 1 "GND" H 10150 2350 50  0000 C CNN
 F 2 "" H 10150 2500 50  0001 C CNN
@@
 $EndComp
 $Comp
-L GND #PWR29
+L GND #PWR020
 U 1 1 5DA63C8C
 P 10600 2550
-F 0 "#PWR29" H 10600 2300 50  0001 C CNN
+F 0 "#PWR020" H 10600 2300 50  0001 C CNN
 F 1 "GND" H 10600 2400 50  0000 C CNN
 F 2 "" H 10600 2550 50  0001 C CNN
@@
 Connection ~ 10600 2450
 $Comp
-L GND #PWR3
+L GND #PWR021
 U 1 1 5DA6715C
 P 900 4450
-F 0 "#PWR3" H 900 4200 50  0001 C CNN
+F 0 "#PWR021" H 900 4200 50  0001 C CNN
 F 1 "GND" H 900 4300 50  0000 C CNN
 F 2 "" H 900 4450 50  0001 C CNN
@@
 	3550 7050 4000 7050
 $Comp
-L GND #PWR9
+L GND #PWR022
 U 1 1 5DA6AF98
 P 2550 7250
-F 0 "#PWR9" H 2550 7000 50  0001 C CNN
+F 0 "#PWR022" H 2550 7000 50  0001 C CNN
 F 1 "GND" H 2550 7100 50  0000 C CNN
 F 2 "" H 2550 7250 50  0001 C CNN
@@
 	3550 6000 4000 6000
 $Comp
-L GND #PWR8
+L GND #PWR023
 U 1 1 5DA6BBF4
 P 2550 6200
-F 0 "#PWR8" H 2550 5950 50  0001 C CNN
+F 0 "#PWR023" H 2550 5950 50  0001 C CNN
 F 1 "GND" H 2550 6050 50  0000 C CNN
 F 2 "" H 2550 6200 50  0001 C CNN
@@
 $EndComp
 $Comp
-L +5V #PWR6
+L +5V #PWR024
 U 1 1 5DA6D8C1
 P 1650 5550
-F 0 "#PWR6" H 1650 5400 50  0001 C CNN
+F 0 "#PWR024" H 1650 5400 50  0001 C CNN
 F 1 "+5V" H 1650 5690 50  0000 C CNN
 F 2 "" H 1650 5550 50  0001 C CNN
@@
 	2200 7050 2050 7050
 $Comp
-L VDDA #PWR5
+L VDDA #PWR025
 U 1 1 5DA6DF11
 P 1300 6800
-F 0 "#PWR5" H 1300 6650 50  0001 C CNN
+F 0 "#PWR025" H 1300 6650 50  0001 C CNN
 F 1 "VDDA" H 1300 6950 50  0000 C CNN
 F 2 "" H 1300 6800 50  0001 C CNN
@@
 $EndComp
 $Comp
-L GND #PWR7
+L GND #PWR026
 U 1 1 5DA6E2C6
 P 1650 7500
-F 0 "#PWR7" H 1650 7250 50  0001 C CNN
+F 0 "#PWR026" H 1650 7250 50  0001 C CNN
 F 1 "GND" H 1650 7350 50  0000 C CNN
 F 2 "" H 1650 7500 50  0001 C CNN
@@
 	2200 6000 2050 6000
 $Comp
-L VDDA #PWR4
+L VDDA #PWR027
 U 1 1 5DA6E2D9
 P 1300 5750
-F 0 "#PWR4" H 1300 5600 50  0001 C CNN
+F 0 "#PWR027" H 1300 5600 50  0001 C CNN
 F 1 "VDDA" H 1300 5900 50  0000 C CNN
 F 2 "" H 1300 5750 50  0001 C CNN
@@
 $EndComp
 $Comp
-L GND #PWR2
+L GND #PWR028
 U 1 1 5DA71E50
 P 850 6800
-F 0 "#PWR2" H 850 6550 50  0001 C CNN
+F 0 "#PWR028" H 850 6550 50  0001 C CNN
 F 1 "GND" H 850 6650 50  0000 C CNN
 F 2 "" H 850 6800 50  0001 C CNN
@@
 $EndComp
 $Comp
-L +5V #PWR1
+L +5V #PWR029
 U 1 1 5DA71E56
 P 850 6200
-F 0 "#PWR1" H 850 6050 50  0001 C CNN
+F 0 "#PWR029" H 850 6050 50  0001 C CNN
 F 1 "+5V" H 850 6340 50  0000 C CNN
 F 2 "" H 850 6200 50  0001 C CNN
@@
 Wire Wire Line
 	1850 3850 1600 3850
-$Comp
-L Conn_01x03 J3
-U 1 1 5DBD7E87
+Wire Wire Line
+	8300 4200 8300 4050
+$Comp
+L Conn_01x04 J3
+U 1 1 5F208D70
 P 8300 3850
-F 0 "J3" V 8400 4000 50  0000 C CNN
-F 1 "UART" V 8400 3750 50  0000 C CNN
-F 2 "Pin_Headers:Pin_Header_Straight_1x03_Pitch2.54mm" H 8300 3850 50  0001 C CNN
+F 0 "J3" V 8400 3975 50  0000 C CNN
+F 1 "UART" V 8400 3700 50  0000 C CNN
+F 2 "Pin_Headers:Pin_Header_Straight_1x04_Pitch2.54mm" H 8300 3850 50  0001 C CNN
 F 3 "" H 8300 3850 50  0001 C CNN
 	1    8300 3850
 	0    -1   -1   0
 $EndComp
-Wire Wire Line
-	8300 4200 8300 4050
+Text Label 6950 4050 2    50   ~ 0
+~RST
+Text Label 8725 4550 2    50   ~ 0
+~RST
+$Comp
+L C C17
+U 1 1 5F20978D
+P 8500 4300
+F 0 "C17" H 8525 4400 50  0000 L CNN
+F 1 "100nF" H 8525 4200 50  0000 L CNN
+F 2 "Capacitors_SMD:C_0805" H 8538 4150 50  0001 C CNN
+F 3 "" H 8500 4300 50  0001 C CNN
+F 4 "Kemet" H 8500 4300 60  0001 C CNN "Manufacturer"
+F 5 "C0805C104J5RACTU" H 8500 4300 60  0001 C CNN "Manufacturer Part Number"
+	1    8500 4300
+	1    0    0    -1
+$EndComp
+Wire Wire Line
+	8500 4050 8500 4150
+Wire Wire Line
+	8500 4450 8500 4550
+Wire Wire Line
+	8500 4550 8725 4550
 $EndSCHEMATC
